Commit message: feature: added plinth for robot

File: ur_description/urdf/ur5_robot.urdf.xacro (robot description, xacro)
@@ -11,9 +11,43 @@
     transmission_hw_interface="$(arg transmission_hw_interface)"
   />
-  <link name="world" />
-  <joint name="world_joint" type="fixed">
-    <parent link="world" />
-    <child link = "base_link" />
-    <origin xyz="0.0 0.0 0.0" rpy="0.0 0.0 0.0" />
-  </joint>
+    <link name="world">
+      <collision>
+        <origin xyz="0 0 0" rpy="0 0 0"/>
+        <geometry>
+           <box size="3 3 0.01"/>
+        </geometry>
+       </collision>
+       <visual>
+         <origin xyz="0 0 0" rpy="0 0 0"/>
+           <geometry>
+             <box size="3 3 0.01"/>
+           </geometry>
+         <material name="blue"/>
+       </visual>
+    </link>
+    <joint name="floor" type="fixed">
+      <parent link="world"/>
+      <child link="plinth_link"/>
+    </joint>
+    <link name="plinth_link">
+      <collision>
+        <origin xyz="0 0 0.4" rpy="0 0 0"/>
+        <geometry>
+           <cylinder radius="0.1" length="0.8"/>
+        </geometry>
+       </collision>
+       <visual>
+         <origin xyz="0 0 0.4" rpy="0 0 0"/>
+           <geometry>
+             <cylinder
+ radius="0.1" length="0.8"/>
+           </geometry>
+         <material name="black"/>
+       </visual>
+    </link>
+    <joint name="plinth" type="fixed">
+      <origin xyz="0.0 0.0 0.81" rpy="0.0 0.0 0.0" />
+      <parent link="plinth_link"/>
+      <child link="base_link"/>
+    </joint>
 </robot>

Commit message: feature: updated impact

File: ur_description/urdf/ur5_robot.urdf.xacro (robot description, xacro)
@@ -23,5 +23,7 @@
              <box size="3 3 0.01"/>
            </geometry>
-         <material name="blue"/>
+         <material name="LightGrey">
+          <color rgba="0.7 0.7 0.7 1.0"/>
+        </material>
        </visual>
     </link>
@@ -32,5 +34,5 @@
     <link name="plinth_link">
       <collision>
-        <origin xyz="0 0 0.4" rpy="0 0 0"/>
+        <origin xyz="0 0 0.402" rpy="0 0 0"/>
         <geometry>
            <cylinder radius="0.1" length="0.8"/>

Commit message: Update xacro as floor collides with plinth

File: ur_description/urdf/ur5_robot.urdf.xacro (robot description, xacro)
@@ -34,5 +34,5 @@
     <link name="plinth_link">
       <collision>
-        <origin xyz="0 0 0.402" rpy="0 0 0"/>
+        <origin xyz="0 0 0.412" rpy="0 0 0"/>
         <geometry>
            <cylinder radius="0.1" length="0.8"/>
